Commit message: third

File: urdf/rasberian.urdf.xacro (robot description, xacro)
@@ -21,9 +21,10 @@
             <material name="silver">
                 <!-- <color rgba="0.75 0.75 0.75 1"/> -->
-                <script>
-                    <uri>/home/ahal/catkin_ws/src/rasberian/model/materials/scripts</uri>
+                <!-- <script>
+                    <uri>/home/ahal/catkin_ws/src/rasberian/model/materials/scripts/marker.material</uri>
                     <uri>/home/ahal/catkin_ws/src/rasberian/model/materials/texture/model.jpg</uri>
                     <name>rasberian/body</name>
-                </script>
+                </script> -->
+                <texture filename="/home/ahal/catkin_ws/src/rasberian/model/materials/scripts/model.jpg" />
             </material>
         </visual>
@@ -85,5 +86,7 @@
         <sphere radius="0.00625"/>
       </geometry>
-      <material name="Black"/>
+        <material name="black">
+             <color rgba="0 0 0 1"/>
+        </material>
     </visual>
     <collision>
@@ -111,10 +114,10 @@
         <collision>
             <geometry>
-                <box size="0.01 0.01 0.01"/>
+                <box size="0.01 0.01 0.04"/>
             </geometry>
         </collision>
         <visual>
             <geometry>
-                <box size="0.01 0.01 0.01"/>
+                <box size="0.01 0.01 0.04"/>
             </geometry>
             <material name="silver">
@@ -126,5 +129,5 @@
         <parent link="base_link"/>
         <child link="caster_support"/>
-        <origin rpy="0 0 0" xyz="0.03 0.0 -0.02825"/>
+        <origin rpy="0 0 0" xyz="0.03 0.0 -0.002"/>
         <!-- <axis xyz="0 0 1"/> -->
     </joint>
@@ -132,10 +135,10 @@
         <parent link="caster_support"/>
         <child link="caster"/>
-        <origin rpy="0 0 0" xyz="0.0 0.0 0"/>
+        <origin rpy="0 0 0" xyz="0.0 0.0 -0.02525"/>
         <axis xyz="0 1 0"/>
     </joint>
     <!-- gazebo -->
     <gazebo reference="base_link">
-        <material>Gazebo/Grey</material>
+        <material>Gazebo/model</material>
         <mu1>0.1</mu1>
         <mu2>0.1</mu2>
@@ -161,3 +164,8 @@
         <mu2>0.1</mu2>
     </gazebo>
+    <gazebo reference="caster">
+        <material>Gazebo/Black</material>
+        <mu1>0.1</mu1>
+        <mu2>0.1</mu2>
+    </gazebo>
 </robot>
